File: biometric access door lock.kicad_sch (KiCad schematic)
At the start: 0 parts

Commit message: update
Parts:
- added J1: R307S, symbol Connector:Conn_01x04_Pin
- added U1: ESP32-WROOM-32, RF_Module:ESP32-WROOM-32, symbol RF_Module:ESP32-WROOM-32
- added U2: LM2596S-5, Package_TO_SOT_SMD:TO-263-5_TabPin3, symbol Regulator_Switching:LM2596S-5
Connections:
- new net: U1.1 (GND), U1.15 (GND), U1.38 (GND), U1.39 (GND)

Commit message: .
Parts:
- removed U2: LM2596S-5, Package_TO_SOT_SMD:TO-263-5_TabPin3, symbol Regulator_Switching:LM2596S-5
- added BZ1: Buzzer, symbol Device:Buzzer
- added D1, D2, D3, D4, D5, D6, D7, D8: SK6812, LED_SMD:LED_SK6812_PLCC4_5.0x5.0mm_P3.2mm, symbol LED:SK6812
- added J2, J3: ~, symbol Connector:Conn_01x03_Pin
- added J4, J5, J6: ~, symbol Connector:Conn_01x02_Pin
- J1: value R307S -> ~
Connections:
- new net: D5.4 (DOUT), D6.2 (DIN)
- new net: D6.4 (DOUT), D7.2 (DIN)
- new net: D1.2 (DIN), D8.4 (DOUT)
- new net: D1.4 (DOUT), D2.2 (DIN)
- new net: D2.4 (DOUT), D3.2 (DIN)
- new net: D3.4 (DOUT), D4.2 (DIN)
- new net: D4.4 (DOUT), D5.2 (DIN)
Other:
- note added: "12V Relay"
- note added: "Buck Converter"
- note added: "Fingerprint Scanner"
- note added: "R307S"
- note added: "Solenoid Door Lock"
- moved on the sheet: J1
